File: meatreader-rev-b/calibration_sensor.kicad_sch (KiCad schematic)
At the start: 5 parts, among them J5 AudioJack3

Commit message: start routing
Parts:
- C13: footprint (none) -> Capacitor_SMD:C_0603_1608Metric
- D8: renamed from D6; footprint (none) -> Diode_SMD:D_0402_1005Metric
- J5: footprint (none) -> Connector_Audio:PJ-320A_TRS
- R18: renamed from R15; footprint (none) -> Resistor_SMD:R_0603_1608Metric
- R19: renamed from R16; footprint (none) -> Resistor_SMD:R_0603_1608Metric
Other:
- title: (none) -> MeatReader Calibration Probe
Changed lines of the file:
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@@
 	(generator "eeschema")
 	(generator_version "9.0")
-	(paper "A4")
+	(paper "USLetter")
+	(title_block
+		(title "MeatReader Calibration Probe")
+		(date "2026-01-17")
+		(rev "B")
+	)
 	(text "External waterproof DS18B20 probe\nDigital 1-Wire temperature sensor"
 		(exclude_from_sim no)
@@
 		(effects
 			(font
-				(size 1.27 1.27)
+				(size 1.524 1.524)
 			)
 		)
@@
 		(on_board yes)
 		(dnp no)
-		(property "Reference" "R15"
+		(property "Reference" "R18"
 			(at 173.736 89.154 90)
 			(effects
@@
 			)
 		)
-		(property "Footprint" ""
+		(property "Footprint" "Resistor_SMD:R_0603_1608Metric"
 			(at 173.99 92.202 90)
 			(effects
@@
 			(project ""
 				(path "/3c2ccb89-2e7f-4bd2-93e9-c6d084b9c33d/b0090d3f-6564-4767-99ad-313e625b5085"
-					(reference "R15")
+					(reference "R18")
 					(unit 1)
 				)
@@
 			)
 		)
-		(property "Footprint" ""
+		(property "Footprint" "Capacitor_SMD:C_0603_1608Metric"
 			(at 162.56 85.09 0)
 			(effects
@@
 			)
 		)
-		(property "Footprint" ""
+		(property "Footprint" "Connector_Audio:PJ-320A_TRS"
 			(at 149.86 93.98 0)
 			(effects
@@
 		(dnp no)
 		(fields_autoplaced yes)
-		(property "Reference" "R16"
+		(property "Reference" "R19"
 			(at 184.15 86.3599 0)
 			(effects
@@
 			)
 		)
-		(property "Footprint" ""
+		(property "Footprint" "Resistor_SMD:R_0603_1608Metric"
 			(at 179.832 87.63 90)
 			(effects
@@
 			(project ""
 				(path "/3c2ccb89-2e7f-4bd2-93e9-c6d084b9c33d/b0090d3f-6564-4767-99ad-313e625b5085"
-					(reference "R16")
+					(reference "R19")
 					(unit 1)
 				)
@@
 		(dnp no)
 		(fields_autoplaced yes)
-		(property "Reference" "#PWR030"
+		(property "Reference" "#PWR022"
 			(at 156.21 104.14 0)
 			(effects
@@
 			(project "meatreader-rev-b"
 				(path "/3c2ccb89-2e7f-4bd2-93e9-c6d084b9c33d/b0090d3f-6564-4767-99ad-313e625b5085"
-					(reference "#PWR030")
+					(reference "#PWR022")
 					(unit 1)
 				)
@@
 		(on_board yes)
 		(dnp no)
-		(property "Reference" "#PWR031"
+		(property "Reference" "#PWR023"
 			(at 162.56 93.98 0)
 			(effects
@@
 			(project "meatreader-rev-b"
 				(path "/3c2ccb89-2e7f-4bd2-93e9-c6d084b9c33d/b0090d3f-6564-4767-99ad-313e625b5085"
-					(reference "#PWR031")
+					(reference "#PWR023")
 					(unit 1)
 				)
@@
 		(dnp no)
 		(fields_autoplaced yes)
-		(property "Reference" "#PWR029"
+		(property "Reference" "#PWR024"
 			(at 162.56 109.22 0)
 			(effects
@@
 			(project ""
 				(path "/3c2ccb89-2e7f-4bd2-93e9-c6d084b9c33d/b0090d3f-6564-4767-99ad-313e625b5085"
-					(reference "#PWR029")
+					(reference "#PWR024")
 					(unit 1)
 				)
@@
 		(dnp no)
 		(fields_autoplaced yes)
-		(property "Reference" "#PWR028"
+		(property "Reference" "#PWR025"
 			(at 181.61 83.82 0)
 			(effects
@@
 			(project ""
 				(path "/3c2ccb89-2e7f-4bd2-93e9-c6d084b9c33d/b0090d3f-6564-4767-99ad-313e625b5085"
-					(reference "#PWR028")
+					(reference "#PWR025")
 					(unit 1)
 				)
@@
 		(dnp no)
 		(fields_autoplaced yes)
-		(property "Reference" "D6"
+		(property "Reference" "D8"
 			(at 165.1 97.7899 90)
 			(effects
@@
 			)
 		)
-		(property "Footprint" ""
+		(property "Footprint" "Diode_SMD:D_0402_1005Metric"
 			(at 162.56 99.06 0)
 			(effects
@@
 			(project ""
 				(path "/3c2ccb89-2e7f-4bd2-93e9-c6d084b9c33d/b0090d3f-6564-4767-99ad-313e625b5085"
-					(reference "D6")
-					(unit 1)
-				)
+					(reference "D8")
+					(unit 1)
+				)
