File: meatreader-rev-b/esp32_core.kicad_sch (KiCad schematic)
At the start: 10 parts, among them U3 ESP32-WROOM-32U

Commit message: start routing
Parts:
- added R7, R9: 4K7, Resistor_SMD:R_0603_1608Metric, symbol Device:R
- C6: renamed from C8; footprint (none) -> Capacitor_SMD:C_0603_1608Metric
- J_UART1: renamed from J_UART; footprint (none) -> Connector_PinHeader_2.54mm:PinHeader_1x04_P2.54mm_Vertical
- SW_BOOT1: renamed from SW_BOOT; footprint (none) -> TestPoint:Test_01x02
- SW_RESET1: renamed from SW_RESET; footprint (none) -> Button_Switch_THT:SW_PUSH_6mm
- U3: value ESP32-WROOM-32U -> ESP32-WROOM-32; footprint RF_Module:ESP32-WROOM-32U -> RF_Module:ESP32-WROOM-32_NoThermals; symbol RF_Module:ESP32-WROOM-32U -> RF_Module:ESP32-WROOM-32
- renumbered C6 to C7, C7 to C8, R5 to R6, R6 to R8
Connections:
- net +3V3: now also R7.1, R9.1
- net ENC_BTN: now reaches U3.10 (IO25)
- net ADC_ALERT: now reaches U3.11 (IO26)
- net CALIB_DATA: now reaches U3.12 (IO27)
- net I2C_SDA: now reaches U3.33 (IO21)
- net I2C_SDA: now also R7.2
- net I2C_SCL: now reaches U3.36 (IO22)
- net I2C_SCL: now also R9.2
- net ENC_A: now reaches U3.8 (IO32)
- net ENC_B: now reaches U3.9 (IO33)
- no-connect marks 0 -> 22
Other:
- note added: "ESP32 Module"
- note added: "I2C Pullups"
- title: (none) -> MeatReader ESP
