File: meatreader-rev-b/meatreader-rev-b.kicad_sch (KiCad schematic)
At the start: 0 parts

Commit message: Power and ESP core
Other:
- added sheet ESP32 Core (esp32_core.kicad_sch)
- added sheet Power (power.kicad_sch)
Changed lines of the file:
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@@
 	(generator_version "9.0")
 	(paper "A4")
+	(global_label "3V3"
+		(shape input)
+		(at 30.48 97.79 180)
+		(fields_autoplaced yes)
+		(effects
+			(font
+				(size 1.27 1.27)
+			)
+			(justify right)
+		)
+		(property "Intersheetrefs" "${INTERSHEET_REFS}"
+			(at 24.5087 97.79 0)
+			(effects
+				(font
+					(size 1.27 1.27)
+				)
+				(justify right)
+				(hide yes)
+			)
+		)
+	)
+	(global_label "BAT"
+		(shape input)
+		(at 30.48 92.71 180)
+		(fields_autoplaced yes)
+		(effects
+			(font
+				(size 1.27 1.27)
+			)
+			(justify right)
+		)
+		(property "Intersheetrefs" "${INTERSHEET_REFS}"
+			(at 24.5087 92.71 0)
+			(effects
+				(font
+					(size 1.27 1.27)
+				)
+				(justify right)
+				(hide yes)
+			)
+		)
+	)
+	(global_label "GND"
+		(shape input)
+		(at 30.48 102.87 180)
+		(fields_autoplaced yes)
+		(effects
+			(font
+				(size 1.27 1.27)
+			)
+			(justify right)
+		)
+		(property "Intersheetrefs" "${INTERSHEET_REFS}"
+			(at 24.5087 102.87 0)
+			(effects
+				(font
+					(size 1.27 1.27)
+				)
+				(justify right)
+				(hide yes)
+			)
+		)
+	)
+	(global_label "VBUS"
+		(shape input)
+		(at 30.48 87.63 180)
+		(fields_autoplaced yes)
+		(effects
+			(font
+				(size 1.27 1.27)
+			)
+			(justify right)
+		)
+		(property "Intersheetrefs" "${INTERSHEET_REFS}"
+			(at 23.4391 87.63 0)
+			(effects
+				(font
+					(size 1.27 1.27)
+				)
+				(justify right)
+				(hide yes)
+			)
+		)
+	)
+	(sheet
+		(at 22.86 20.32)
+		(size 74.93 44.45)
+		(exclude_from_sim no)
+		(in_bom yes)
+		(on_board yes)
+		(dnp no)
+		(fields_autoplaced yes)
+		(stroke
+			(width 0.1524)
+			(type solid)
+		)
+		(fill
+			(color 0 0 0 0.0000)
+		)
+		(property "Sheetname" "Power"
+			(at 22.86 19.6084 0)
+			(effects
+				(font
+					(size 1.27 1.27)
+				)
+				(justify left bottom)
+			)
+		)
+		(property "Sheetfile" "power.kicad_sch"
+			(at 22.86 65.3546 0)
+			(effects
+				(font
+					(size 1.27 1.27)
+				)
+				(justify left top)
+			)
+		)
+		(instances
+			(project "meatreader-rev-b"
+				(path "/3c2ccb89-2e7f-4bd2-93e9-c6d084b9c33d"
+					(page "2")
+				)
+			)
+		)
+	)
+	(sheet
+		(at 106.68 20.32)
+		(size 86.36 44.45)
+		(exclude_from_sim no)
+		(in_bom yes)
+		(on_board yes)
+		(dnp no)
+		(fields_autoplaced yes)
+		(stroke
+			(width 0.1524)
+			(type solid)
+		)
+		(fill
+			(color 0 0 0 0.0000)
+		)
+		(property "Sheetname" "ESP32 Core"
+			(at 106.68 19.6084 0)
+			(effects
+				(font
+					(size 1.27 1.27)
+				)
+				(justify left bottom)
+			)
+		)
+		(property "Sheetfile" "esp32_core.kicad_sch"
+			(at 106.68 65.3546 0)
+			(effects
+				(font
+					(size 1.27 1.27)
+				)
+				(justify left top)
+			)
+		)
+		(instances
+			(project "meatreader-rev-b"
+				(path "/3c2ccb89-2e7f-4bd2-93e9-c6d084b9c33d"
+					(page "3")
+				)
+			)
+		)
+	)
 	(sheet_instances
 		(path "/"

Commit message: rev-b initial commit
Other:
- added sheet Calibration Sensor (calibration_sensor.kicad_sch)
- added sheet Sensors ADC (sensors_adc.kicad_sch)
- added sheet UI (ui.kicad_sch)
Changed lines of the file:
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@@
 	(generator_version "9.0")
 	(paper "A4")
+	(global_label "I2C_SDA"
+		(shape input)
+		(at 63.5 73.66 180)
+		(fields_autoplaced yes)
+		(effects
+			(font
+				(size 1.27 1.27)
+			)
+			(justify right)
+		)
+		(property "Intersheetrefs" "${INTERSHEET_REFS}"
+			(at 53.2505 73.66 0)
+			(effects
+				(font
+					(size 1.27 1.27)
+				)
+				(justify right)
+				(hide yes)
+			)
+		)
+	)
+	(global_label "I2C_SCL"
+		(shape input)
+		(at 63.5 78.74 180)
+		(fields_autoplaced yes)
+		(effects
+			(font
+				(size 1.27 1.27)
+			)
+			(justify right)
+		)
+		(property "Intersheetrefs" "${INTERSHEET_REFS}"
+			(at 53.2505 78.74 0)
+			(effects
+				(font
+					(size 1.27 1.27)
+				)
+				(justify right)
+				(hide yes)
+			)
+		)
+	)
 	(global_label "3V3"
 		(shape input)
-		(at 30.48 97.79 180)
-		(fields_autoplaced yes)
-		(effects
-			(font
-				(size 1.27 1.27)
-			)
-			(justify right)
-		)
-		(property "Intersheetrefs" "${INTERSHEET_REFS}"
-			(at 24.5087 97.79 0)
+		(at 63.5 63.5 180)
+		(fields_autoplaced yes)
+		(effects
+			(font
+				(size 1.27 1.27)
+			)
+			(justify right)
+		)
+		(property "Intersheetrefs" "${INTERSHEET_REFS}"
+			(at 57.5287 63.5 0)
 			(effects
 				(font
@@
 	(global_label "BAT"
 		(shape input)
-		(at 30.48 92.71 180)
-		(fields_autoplaced yes)
-		(effects
-			(font
-				(size 1.27 1.27)
-			)
-			(justify right)
-		)
-		(property "Intersheetrefs" "${INTERSHEET_REFS}"
-			(at 24.5087 92.71 0)
+		(at 63.5 58.42 180)
+		(fields_autoplaced yes)
+		(effects
+			(font
+				(size 1.27 1.27)
+			)
+			(justify right)
+		)
+		(property "Intersheetrefs" "${INTERSHEET_REFS}"
+			(at 57.5287 58.42 0)
 			(effects
 				(font
@@
 	(global_label "GND"
 		(shape input)
-		(at 30.48 102.87 180)
-		(fields_autoplaced yes)
-		(effects
-			(font
-				(size 1.27 1.27)
-			)
-			(justify right)
-		)
-		(property "Intersheetrefs" "${INTERSHEET_REFS}"
-			(at 24.5087 102.87 0)
+		(at 63.5 68.58 180)
+		(fields_autoplaced yes)
+		(effects
+			(font
+				(size 1.27 1.27)
+			)
+			(justify right)
+		)
+		(property "Intersheetrefs" "${INTERSHEET_REFS}"
+			(at 57.5287 68.58 0)
+			(effects
+				(font
+					(size 1.27 1.27)
+				)
+				(justify right)
+				(hide yes)
+			)
+		)
+	)
+	(global_label "ADC_ALERT"
+		(shape input)
+		(at 63.5 83.82 180)
+		(fields_autoplaced yes)
+		(effects
+			(font
+				(size 1.27 1.27)
+			)
+			(justify right)
+		)
+		(property "Intersheetrefs" "${INTERSHEET_REFS}"
+			(at 51.1115 83.82 0)
 			(effects
 				(font
@@
 	(global_label "VBUS"
 		(shape input)
-		(at 30.48 87.63 180)
-		(fields_autoplaced yes)
-		(effects
-			(font
-				(size 1.27 1.27)
-			)
-			(justify right)
-		)
-		(property "Intersheetrefs" "${INTERSHEET_REFS}"
-			(at 23.4391 87.63 0)
-			(effects
-				(font
-					(size 1.27 1.27)
-				)
-				(justify right)
-				(hide yes)
-			)
-		)
-	)
-	(sheet
-		(at 22.86 20.32)
-		(size 74.93 44.45)
+		(at 63.5 53.34 180)
+		(fields_autoplaced yes)
+		(effects
+			(font
+				(size 1.27 1.27)
+			)
+			(justify right)
+		)
+		(property "Intersheetrefs" "${INTERSHEET_REFS}"
+			(at 56.4591 53.34 0)
+			(effects
+				(font
+					(size 1.27 1.27)
+				)
+				(justify right)
+				(hide yes)
+			)
+		)
+	)
+	(sheet
+		(at 77.47 20.32)
+		(size 39.37 12.7)
+		(exclude_from_sim no)
+		(in_bom yes)
+		(on_board yes)
+		(dnp no)
+		(fields_autoplaced yes)
+		(stroke
+			(width 0.1524)
+			(type solid)
+		)
+		(fill
+			(color 0 0 0 0.0000)
+		)
+		(property "Sheetname" "Sensors ADC"
+			(at 77.47 19.6084 0)
+			(effects
+				(font
+					(size 1.27 1.27)
+				)
+				(justify left bottom)
+			)
+		)
+		(property "Sheetfile" "sensors_adc.kicad_sch"
+			(at 77.47 33.6046 0)
+			(effects
+				(font
+					(size 1.27 1.27)
+				)
+				(justify left top)
+			)
+		)
+		(instances
+			(project "meatreader-rev-b"
+				(path "/3c2ccb89-2e7f-4bd2-93e9-c6d084b9c33d"
+					(page "4")
+				)
+			)
+		)
+	)
+	(sheet
+		(at 31.75 20.32)
+		(size 39.37 12.7)
 		(exclude_from_sim no)
 		(in_bom yes)
@@
 		)
 		(property "Sheetname" "Power"
-			(at 22.86 19.6084 0)
+			(at 31.75 19.6084 0)
 			(effects
 				(font
@@
 		)
 		(property "Sheetfile" "power.kicad_sch"
-			(at 22.86 65.3546 0)
+			(at 31.75 33.6046 0)
 			(effects
 				(font
@@
 	)
 	(sheet
-		(at 106.68 20.32)
-		(size 86.36 44.45)
+		(at 170.18 20.32)
+		(size 40.64 12.7)
+		(exclude_from_sim no)
+		(in_bom yes)
+		(on_board yes)
+		(dnp no)
+		(fields_autoplaced yes)
+		(stroke
+			(width 0.1524)
+			(type solid)
+		)
+		(fill
+			(color 0 0 0 0.0000)
+		)
+		(property "Sheetname" "UI"
+			(at 170.18 19.6084 0)
+			(effects
+				(font
+					(size 1.27 1.27)
+				)
+				(justify left bottom)
+			)
+		)
+		(property "Sheetfile" "ui.kicad_sch"
+			(at 170.18 33.6046 0)
+			(effects
+				(font
+					(size 1.27 1.27)
+				)
+				(justify left top)
+			)
+		)
+		(instances
+			(project "meatreader-rev-b"
+				(path "/3c2ccb89-2e7f-4bd2-93e9-c6d084b9c33d"
+					(page "6")
+				)
+			)
+		)
+	)
+	(sheet
+		(at 77.47 49.53)
+		(size 46.99 25.4)
 		(exclude_from_sim no)
 		(in_bom yes)
@@
 		)
 		(property "Sheetname" "ESP32 Core"
-			(at 106.68 19.6084 0)
+			(at 77.47 48.8184 0)
 			(effects
 				(font
@@
 		)
 		(property "Sheetfile" "esp32_core.kicad_sch"
-			(at 106.68 65.3546 0)
+			(at 77.47 75.5146 0)
 			(effects
 				(font
@@
 				)
 			)
+		)
+	)
+	(sheet
+		(at 123.19 20.32)
+		(size 39.37 12.7)
+		(exclude_from_sim no)
+		(in_bom yes)
+		(on_board yes)
+		(dnp no)
+		(fields_autoplaced yes)
+		(stroke
+			(width 0.1524)
+			(type solid)
+		)
+		(fill
+			(color 0 0 0 0.0000)
+		)
+		(property "Sheetname" "Calibration Sensor"
+			(at 123.19 19.6084 0)
+			(effects
+				(font
+					(size 1.27 1.27)
+				)
+				(justify left bottom)
+			)
+		)
+		(property "Sheetfile" "calibration_sensor.kicad_sch"
+			(at 123.19 33.6046 0)
+			(effects
+				(font
+					(size 1.27 1.27)
+				)
+				(justify left top)
+			)
+		)
+		(instances
+			(project "meatreader-rev-b"
+				(path "/3c2ccb89-2e7f-4bd2-93e9-c6d084b9c33d"
+					(page "5")
+				)
+			)

Commit message: start routing
Other:
- note added: "ADS1115 + probes"
- note added: "Battery, charger, regulation"
- note added: "DS18B20 calibration"
- note added: "MCU, UART, reset, I/O"
- note added: "OLED + encoder"
- title: (none) -> MeatReader
Changed lines of the file:
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@@
 	(generator "eeschema")
 	(generator_version "9.0")
-	(paper "A4")
-	(global_label "I2C_SDA"
-		(shape input)
-		(at 63.5 73.66 180)
-		(fields_autoplaced yes)
-		(effects
-			(font
-				(size 1.27 1.27)
-			)
-			(justify right)
-		)
-		(property "Intersheetrefs" "${INTERSHEET_REFS}"
-			(at 53.2505 73.66 0)
-			(effects
-				(font
-					(size 1.27 1.27)
-				)
-				(justify right)
-				(hide yes)
-			)
-		)
-	)
-	(global_label "I2C_SCL"
-		(shape input)
-		(at 63.5 78.74 180)
-		(fields_autoplaced yes)
-		(effects
-			(font
-				(size 1.27 1.27)
-			)
-			(justify right)
-		)
-		(property "Intersheetrefs" "${INTERSHEET_REFS}"
-			(at 53.2505 78.74 0)
-			(effects
-				(font
-					(size 1.27 1.27)
-				)
-				(justify right)
-				(hide yes)
-			)
-		)
-	)
-	(global_label "3V3"
-		(shape input)
-		(at 63.5 63.5 180)
-		(fields_autoplaced yes)
-		(effects
-			(font
-				(size 1.27 1.27)
-			)
-			(justify right)
-		)
-		(property "Intersheetrefs" "${INTERSHEET_REFS}"
-			(at 57.5287 63.5 0)
-			(effects
-				(font
-					(size 1.27 1.27)
-				)
-				(justify right)
-				(hide yes)
-			)
-		)
-	)
-	(global_label "BAT"
-		(shape input)
-		(at 63.5 58.42 180)
-		(fields_autoplaced yes)
-		(effects
-			(font
-				(size 1.27 1.27)
-			)
-			(justify right)
-		)
-		(property "Intersheetrefs" "${INTERSHEET_REFS}"
-			(at 57.5287 58.42 0)
-			(effects
-				(font
-					(size 1.27 1.27)
-				)
-				(justify right)
-				(hide yes)
-			)
-		)
-	)
-	(global_label "GND"
-		(shape input)
-		(at 63.5 68.58 180)
-		(fields_autoplaced yes)
-		(effects
-			(font
-				(size 1.27 1.27)
-			)
-			(justify right)
-		)
-		(property "Intersheetrefs" "${INTERSHEET_REFS}"
-			(at 57.5287 68.58 0)
-			(effects
-				(font
-					(size 1.27 1.27)
-				)
-				(justify right)
-				(hide yes)
-			)
-		)
-	)
-	(global_label "ADC_ALERT"
-		(shape input)
-		(at 63.5 83.82 180)
-		(fields_autoplaced yes)
-		(effects
-			(font
-				(size 1.27 1.27)
-			)
-			(justify right)
-		)
-		(property "Intersheetrefs" "${INTERSHEET_REFS}"
-			(at 51.1115 83.82 0)
-			(effects
-				(font
-					(size 1.27 1.27)
-				)
-				(justify right)
-				(hide yes)
-			)
-		)
-	)
-	(global_label "VBUS"
-		(shape input)
-		(at 63.5 53.34 180)
-		(fields_autoplaced yes)
-		(effects
-			(font
-				(size 1.27 1.27)
-			)
-			(justify right)
-		)
-		(property "Intersheetrefs" "${INTERSHEET_REFS}"
-			(at 56.4591 53.34 0)
-			(effects
-				(font
-					(size 1.27 1.27)
-				)
-				(justify right)
-				(hide yes)
-			)
-		)
-	)
-	(sheet
-		(at 77.47 20.32)
-		(size 39.37 12.7)
+	(paper "USLetter")
+	(title_block
+		(title "MeatReader")
+		(date "2026-01-17")
+		(rev "B")
+	)
+	(text "MCU, UART, reset, I/O"
+		(exclude_from_sim no)
+		(at 93.726 108.458 0)
+		(effects
+			(font
+				(size 1.27 1.27)
+			)
+		)
+	)
+	(text "ADS1115 + probes"
+		(exclude_from_sim no)
+		(at 144.78 107.696 0)
+		(effects
+			(font
+				(size 1.27 1.27)
+			)
+		)
+	)
+	(text "OLED + encoder"
+		(exclude_from_sim no)
+		(at 233.68 108.204 0)
+		(effects
+			(font
+				(size 1.27 1.27)
+			)
+		)
+	)
+	(text "Battery, charger, regulation"
+		(exclude_from_sim no)
+		(at 42.164 108.458 0)
+		(effects
+			(font
+				(size 1.27 1.27)
+			)
+		)
+	)
+	(text "DS18B20 calibration"
+		(exclude_from_sim no)
+		(at 189.992 107.95 0)
+		(effects
+			(font
+				(size 1.27 1.27)
+			)
+		)
+	)
+	(sheet
+		(at 128.27 90.17)
+		(size 34.29 33.02)
 		(exclude_from_sim no)
 		(in_bom yes)
@@
 		)
 		(property "Sheetname" "Sensors ADC"
-			(at 77.47 19.6084 0)
+			(at 128.27 89.4584 0)
 			(effects
 				(font
@@
 		)
 		(property "Sheetfile" "sensors_adc.kicad_sch"
-			(at 77.47 33.6046 0)
+			(at 128.27 123.7746 0)
 			(effects
 				(font
@@
 	)
 	(sheet
-		(at 31.75 20.32)
-		(size 39.37 12.7)
+		(at 25.4 91.44)
+		(size 34.29 33.02)
 		(exclude_from_sim no)
 		(in_bom yes)
@@
 		)
 		(property "Sheetname" "Power"
-			(at 31.75 19.6084 0)
+			(at 25.4 90.7284 0)
 			(effects
 				(font
@@
 		)
 		(property "Sheetfile" "power.kicad_sch"
-			(at 31.75 33.6046 0)
+			(at 25.4 125.0446 0)
 			(effects
 				(font
@@
 	)
 	(sheet
-		(at 170.18 20.32)
-		(size 40.64 12.7)
+		(at 215.9 90.17)
+		(size 34.29 33.02)
 		(exclude_from_sim no)
 		(in_bom yes)
@@
 		)
 		(property "Sheetname" "UI"
-			(at 170.18 19.6084 0)
+			(at 215.9 89.4584 0)
 			(effects
 				(font
@@
 		)
 		(property "Sheetfile" "ui.kicad_sch"
-			(at 170.18 33.6046 0)
+			(at 215.9 123.7746 0)
 			(effects
 				(font
@@
 	)
 	(sheet
-		(at 77.47 49.53)
-		(size 46.99 25.4)
+		(at 69.85 85.09)
+		(size 48.26 45.72)
 		(exclude_from_sim no)
 		(in_bom yes)
@@
 		)
 		(property "Sheetname" "ESP32 Core"
-			(at 77.47 48.8184 0)
+			(at 69.85 84.3784 0)
 			(effects
 				(font
@@
 		)
 		(property "Sheetfile" "esp32_core.kicad_sch"
-			(at 77.47 75.5146 0)
+			(at 69.85 131.3946 0)
 			(effects
 				(font
@@
 	)
 	(sheet
-		(at 123.19 20.32)
-		(size 39.37 12.7)
+		(at 172.72 90.17)
+		(size 34.29 33.02)
 		(exclude_from_sim no)
 		(in_bom yes)
@@
 		)
 		(property "Sheetname" "Calibration Sensor"
-			(at 123.19 19.6084 0)
+			(at 172.72 89.4584 0)
 			(effects
 				(font
@@
 		)
 		(property "Sheetfile" "calibration_sensor.kicad_sch"
-			(at 123.19 33.6046 0)
-			(effects
-				(font
+			(at 172.72 123.7746 0)
+			(effects
+				(font
