File: meatreader-rev-b/power.kicad_sch (KiCad schematic)
At the start: 15 parts, among them J1 USB_C_Receptacle_PowerOnly_6P, J2 JST-PH-2, Q1 AO3401A, U1 TP4056-42-ESOP8, U2 AP7361C-33E

Commit message: start routing
Parts:
- removed F1: RXE090, TerminalBlock_Phoenix:TerminalBlock_Phoenix_MKDS-1,5-2-5.08_1x02_P5.08mm_Horizontal, symbol Device:Polyfuse
- removed Q1: AO3401A, Package_TO_SOT_SMD:SOT-23, symbol Transistor_FET:Q_PMOS_GSD
- added D2: LED_G, LED_THT:LED_D3.0mm, symbol Device:LED
- added D3: LED_R, LED_THT:LED_D3.0mm, symbol Device:LED
- added R4: 1K, Resistor_SMD:R_0402_1005Metric, symbol Device:R
- added SW_POWER1: SPST, Connector_PinHeader_2.54mm:PinHeader_1x02_P2.54mm_Vertical, symbol Switch:SW_SPST
- C1: renamed from C3; footprint (none) -> Capacitor_SMD:C_0805_2012Metric
- C2: renamed from C4; footprint (none) -> Capacitor_SMD:C_0805_2012Metric
- C3: renamed from C1; footprint Capacitor_SMD:C_0603_1608Metric -> Capacitor_SMD:C_0805_2012Metric
- C4: renamed from C2; footprint Capacitor_SMD:C_0603_1608Metric -> Capacitor_SMD:C_0805_2012Metric
- D1: value TVS 5V -> SMF5.0A; footprint Package_TO_SOT_SMD:SOT-23 -> Diode_SMD:D_SMF; symbol Device:D_TVS -> Diode:SMF5V0A; LCSC (none) -> C19077497
- R1, R2: footprint Resistor_SMD:R_0603_1608Metric -> Resistor_SMD:R_0402_1005Metric
- R3: value 100K -> 1K; footprint Resistor_SMD:R_0603_1608Metric -> Resistor_SMD:R_0402_1005Metric; LCSC (none) -> C11702
- R5: renamed from R4; footprint Resistor_SMD:R_0603_1608Metric -> Resistor_SMD:R_0402_1005Metric
- U2: renamed from U1; footprint Package_SO:SOIC-8-1EP_3.9x4.9mm_P1.27mm_EP2.41x3.3mm_ThermalVias -> Package_SO:SOIC-8-1EP_3.9x4.9mm_P1.27mm_EP2.41x3.3mm
- renumbered U2 to U1
Connections:
- net BAT: now also J2.1 (Pin_1), SW_POWER1.1 (A); no longer C1.1, U1.1 (VI)
- net GND: no longer R3.2
- net STDBY_LED: now reaches U2.6 (~{STDBY})
- net STDBY_LED: now also R3.1
- net CHARGE_LED: now reaches U2.7 (~{CHRG})
- net CHARGE_LED: now also R4.1
- net VBUS renamed 5V_USB
- net 5V_USB: now also D2.2 (A), D3.2 (A)
- new net: D2.1 (K), R3.2
- new net: D3.1 (K), R4.2
- new net BAT_SYS: C1.1, SW_POWER1.2 (B), U1.1 (VI)
Other:
- note added: "Don't run thin traces for battery current"
- note removed: "Place PTC + PFET right next to battery connector Keep Source ↔ Drain copper short and wide Gate resistor right next to the gate pin Don't run thin traces for battery current"
- title: (none) -> MeatReader Power
- moved on the sheet: C3, C4, R5, U2
