File: meatreader-rev-b/sensors_adc.kicad_sch (KiCad schematic)
At the start: 19 parts, among them J3 2.5MM TS_Jack, J4 2.5MM TS_Jack, U4 ADS1115

Commit message: start routing
Parts:
- C12: renamed from C10; footprint (none) -> Capacitor_SMD:C_0603_1608Metric
- D4: renamed from D2; value H3V3L06B -> D_ESD_SIG; footprint Diode_SMD:D_0201_0603Metric -> Diode_SMD:D_0402_1005Metric
- D5: renamed from D4; value H3V3L06B -> D_ESD_SIG; footprint Diode_SMD:D_0201_0603Metric -> Diode_SMD:D_0402_1005Metric
- D6: renamed from D3; value H3V3L06B -> D_ESD_SIG; footprint (none) -> Diode_SMD:D_0402_1005Metric
- D7: renamed from D5; value H3V3L06B -> D_ESD_SIG; footprint (none) -> Diode_SMD:D_0402_1005Metric
- J3, J4: footprint (none) -> Connector_Audio:Jack_2.5MM_PJ210B_TS; JLC_3DModel_Q (none) -> 9e36057968d7478ca8658f227985305d; JLC_3D_Size (none) -> 5.1 11.225
- R10: renamed from R7; footprint (none) -> Resistor_SMD:R_0603_1608Metric
- R11: renamed from R8; footprint (none) -> Resistor_SMD:R_0603_1608Metric
- R12: renamed from R11; footprint (none) -> Resistor_SMD:R_0603_1608Metric
- R13: renamed from R12; footprint (none) -> Resistor_SMD:R_0603_1608Metric
- R14: renamed from R9; footprint (none) -> Resistor_SMD:R_0603_1608Metric
- R15: renamed from R10; footprint (none) -> Resistor_SMD:R_0603_1608Metric
- R16: renamed from R13; footprint (none) -> Resistor_SMD:R_0603_1608Metric
- R17: renamed from R14; footprint (none) -> Resistor_SMD:R_0603_1608Metric
- renumbered C12 to C10, C9 to C11, C11 to C9
Other:
- note added: "ADS1115 Analog Digital Converter"
- title: (none) -> MeatReader ADC Probes
- moved on the sheet: C11, C12, U4
