File: meatreader-rev-b/ui.kicad_sch (KiCad schematic)
At the start: 4 parts, among them J6 OLED_CONN, J7 ENC_CONN

Commit message: start routing
Parts:
- C14: renamed from C15; footprint (none) -> Capacitor_SMD:C_0603_1608Metric
- C15: renamed from C14; footprint (none) -> Capacitor_SMD:C_0603_1608Metric
- J6: footprint (none) -> Connector_JST:JST_XH_B4B-XH-AM_1x04_P2.50mm_Vertical
- J7: footprint (none) -> Connector_JST:JST_XH_B5B-XH-AM_1x05_P2.50mm_Vertical
Connections:
- net UI_ENC_A renamed ENC_A
- net UI_ENC_B renamed ENC_B
- net UI_ENC_BTN renamed ENC_BTN
Other:
- title: (none) -> MeatReader UI
- moved on the sheet: C14, C15, J6, J7
